File: KiCad/DAC_Vref_IOEXP_Temp.kicad_sch (KiCad schematic)
At the start: 29 parts, among them IC10 PCAL9722HNMP, IC6 DAC8552IDGKR, IC7 74AUP1G74DC,125, IC8 REF5025AIDR, IC9 TC77-5.0MCTTR, Q1 BSS84, Q2 BSS84, Q3 BSS84

Commit message: r4B3 version: OE fixed, new LEDs for remote programming
Parts:
- added JP5: ~, PCM_EEZ_connectors:M22-2010246, symbol PCM_EEZ_unsorted:JP2 open 2mm THT
- added R18: 100K, PCM_EEZ_passives:R_0805_2012Metric, symbol PCM_EEZ_passives:R-EU
- JP4: symbol PCM_EEZ_unsorted:JP2 open -> PCM_EEZ_unsorted:JP2 open 2mm THT; DigiKey 952-3309-ND -> M22-2010346-ND; TME ZL303-02P -> -; now in the parts list
- R24: renamed from R19; Mouser 71-CRCW0805750RFKEB -> 71-CRCW0805750RFKEAC
- renumbered C30 to C33, C31 to C34, C32 to C35, C33 to C39, C34 to C42, C35 to C44, C36 to C47, C37 to C48, C38 to C50, IC9 to IC10, IC10 to IC13, IC8 to IC9, R18 to R22, R20 to R25, R21 to R28, R22 to R33, R23 to R34
Connections:
- net +3V3: now also JP4.1, JP5.1; no longer JP4.2
- net GND: now also R18.1
- net ISO_OE_SYNC: now also JP5.2, R18.2
- net OE_TRIG: now also JP4.2; no longer JP4.1
- net POST_OE: now also IC7.3 (~{Q}); no longer IC7.5 (Q)
- net PREG_OE: now reaches IC13.14 (P1_5)
- no-connect marks 5 -> 4
Other:
- moved on the sheet: C39, D2, D3, IC7A, IC7B, R22, TP1

Commit message: Temp sensor SPI fixed
Connections:
- net ISO_DA_SCLK: now also IC10.3 (SCLK)
- net ISO_IOEXP_MISO: no longer IC10.4 (SI/O)
- net ISO_IOEXP_SCLK: no longer IC10.3 (SCLK)
- new net ISO_DA_MISO: IC10.4 (SI/O)
Changed lines of the file:
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@@
 	(title_block
 		(title "${project_name}")
-		(date "2025-11-27")
+		(date "2025-12-05")
 		(rev "${project_version}")
 		(company "${project_creator}")
@@
 		)
 	)
-	(global_label "~{OVP_FAULT}"
-		(shape input)
-		(at 27.94 101.6 180)
+	(global_label "ISO_DA_MISO"
+		(shape output)
+		(at 124.46 149.86 180)
 		(fields_autoplaced yes)
 		(effects
@@
 		)
 		(property "Intersheetrefs" "${INTERSHEET_REFS}"
-			(at 18.7386 101.6 0)
+			(at 113.9463 149.86 0)
 			(effects
 				(font
@@
 		)
 	)
+	(global_label "~{OVP_FAULT}"
+		(shape input)
+		(at 27.94 101.6 180)
+		(fields_autoplaced yes)
+		(effects
+			(font
+				(size 0.889 0.889)
+			)
+			(justify right)
+		)
+		(property "Intersheetrefs" "${INTERSHEET_REFS}"
+			(at 18.7386 101.6 0)
+			(effects
+				(font
+					(size 1.27 1.27)
+				)
+				(justify right)
+				(hide yes)
+			)
+		)
+	)
 	(global_label "I_SET"
 		(shape output)
@@
 		)
 	)
-	(global_label "ISO_IOEXP_SCLK"
+	(global_label "PREG_OE"
+		(shape output)
+		(at 243.84 68.58 0)
+		(fields_autoplaced yes)
+		(effects
+			(font
+				(size 0.889 0.889)
+			)
+			(justify left)
+		)
+		(property "Intersheetrefs" "${INTERSHEET_REFS}"
+			(at 251.8137 68.58 0)
+			(effects
+				(font
+					(size 1.27 1.27)
+				)
+				(justify left)
+				(hide yes)
+			)
+		)
+	)
+	(global_label "ISO_DA_SCLK"
 		(shape input)
 		(at 124.46 147.32 180)
@@
 		)
 		(property "Intersheetrefs" "${INTERSHEET_REFS}"
-			(at 111.5756 147.32 0)
+			(at 113.8192 147.32 0)
 			(effects
 				(font
@@
 		)
 	)
-	(global_label "PREG_OE"
-		(shape output)
-		(at 243.84 68.58 0)
-		(fields_autoplaced yes)
-		(effects
-			(font
-				(size 0.889 0.889)
-			)
-			(justify left)
-		)
-		(property "Intersheetrefs" "${INTERSHEET_REFS}"
-			(at 251.8137 68.58 0)
-			(effects
-				(font
-					(size 1.27 1.27)
-				)
-				(justify left)
-				(hide yes)
-			)
-		)
-	)
 	(global_label "~{ISO_IOEXP_IRQ}"
 		(shape output)
@@
 			(effects
 				(font
-					(size 1.27 1.27)
-				)
-				(justify right)
-				(hide yes)
-			)
-		)
-	)
-	(global_label "ISO_IOEXP_MISO"
-		(shape output)
-		(at 124.46 149.86 180)
-		(fields_autoplaced yes)
-		(effects
-			(font
-				(size 0.889 0.889)
-			)
-			(justify right)
-		)
-		(property "Intersheetrefs" "${INTERSHEET_REFS}"
-			(at 111.7027 149.86 0)
-			(effects
-				(font

Commit message: EEPROM connected to H503 I2C bus
Parts:
- renumbered JP4 to JP2, JP5 to JP3, R18 to R15, R22 to R19, R24 to R21, R25 to R22, R28 to R25, R33 to R30, R34 to R31
Changed lines of the file:
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@@
 	(title_block
 		(title "${project_name}")
-		(date "2025-12-05")
+		(date "2025-12-06")
 		(rev "${project_version}")
 		(company "${project_creator}")
@@
 		(on_board yes)
 		(dnp no)
-		(property "Reference" "R24"
+		(property "Reference" "R21"
 			(at 73.66 156.21 90)
 			(effects
@@
 			(project "EEZ DIB2 DCP426"
 				(path "/65943c0e-8943-4d2a-93dc-fb4938f73312/bbd8d1a5-9776-495b-aec4-035cc25cf688"
-					(reference "R24")
+					(reference "R21")
 					(unit 1)
 				)
@@
 		(on_board yes)
 		(dnp no)
-		(property "Reference" "R25"
+		(property "Reference" "R22"
 			(at 73.66 163.83 90)
 			(effects
@@
 			(project "EEZ DIB DCP405plus"
 				(path "/65943c0e-8943-4d2a-93dc-fb4938f73312/bbd8d1a5-9776-495b-aec4-035cc25cf688"
-					(reference "R25")
+					(reference "R22")
 					(unit 1)
 				)
@@
 		(on_board yes)
 		(dnp no)
-		(property "Reference" "R22"
+		(property "Reference" "R19"
 			(at 44.45 83.82 0)
 			(effects
@@
 			(project "EEZ DIB2 DCP426"
 				(path "/65943c0e-8943-4d2a-93dc-fb4938f73312/bbd8d1a5-9776-495b-aec4-035cc25cf688"
-					(reference "R22")
+					(reference "R19")
 					(unit 1)
 				)
@@
 		(on_board yes)
 		(dnp no)
-		(property "Reference" "R28"
+		(property "Reference" "R25"
 			(at 123.19 80.01 0)
 			(effects
@@
 			(project "EEZ DIB2 DCP426"
 				(path "/65943c0e-8943-4d2a-93dc-fb4938f73312/bbd8d1a5-9776-495b-aec4-035cc25cf688"
-					(reference "R28")
+					(reference "R25")
 					(unit 1)
 				)
@@
 		(on_board yes)
 		(dnp no)
-		(property "Reference" "R33"
+		(property "Reference" "R30"
 			(at 139.7 97.79 90)
 			(effects
@@
 			(project "EEZ DIB2 DCP426"
 				(path "/65943c0e-8943-4d2a-93dc-fb4938f73312/bbd8d1a5-9776-495b-aec4-035cc25cf688"
-					(reference "R33")
+					(reference "R30")
 					(unit 1)
 				)
@@
 		(on_board yes)
 		(dnp yes)
-		(property "Reference" "JP5"
+		(property "Reference" "JP3"
 			(at 40.64 77.47 0)
 			(effects
@@
 			(project "EEZ DIB DCP405plus"
 				(path "/65943c0e-8943-4d2a-93dc-fb4938f73312/bbd8d1a5-9776-495b-aec4-035cc25cf688"
-					(reference "JP5")
+					(reference "JP3")
 					(unit 1)
 				)
@@
 		(on_board yes)
 		(dnp no)
-		(property "Reference" "R34"
+		(property "Reference" "R31"
 			(at 205.74 34.29 90)
 			(effects
@@
 			(project "EEZ DIB2 DCP426"
 				(path "/65943c0e-8943-4d2a-93dc-fb4938f73312/bbd8d1a5-9776-495b-aec4-035cc25cf688"
-					(reference "R34")
+					(reference "R31")
 					(unit 1)
 				)
@@
 		(on_board yes)
 		(dnp no)
-		(property "Reference" "R18"
+		(property "Reference" "R15"
 			(at 30.48 74.93 90)
 			(effects
@@
 			(project "EEZ DIB DCP405plus"
 				(path "/65943c0e-8943-4d2a-93dc-fb4938f73312/bbd8d1a5-9776-495b-aec4-035cc25cf688"
-					(reference "R18")
+					(reference "R15")
 					(unit 1)
 				)
@@
 		(on_board yes)
 		(dnp yes)
-		(property "Reference" "JP4"
+		(property "Reference" "JP2"
 			(at 38.1 115.57 0)
 			(effects
@@
 			(project "EEZ DIB DCP405plus"
 				(path "/65943c0e-8943-4d2a-93dc-fb4938f73312/bbd8d1a5-9776-495b-aec4-035cc25cf688"
-					(reference "JP4")
+					(reference "JP2")
 					(unit 1)
 				)

Commit message: Vref tantalum capacitor removed
Parts:
- removed C42: 4u7 tant., PCM_EEZ_passives:EC1206, symbol PCM_EEZ_passives:ECAP
- added C41: 22u, PCM_EEZ_passives:C_1210_3225Metric, symbol PCM_EEZ_passives:C-EU
- added C44: 1u, PCM_EEZ_passives:C_0805_2012Metric, symbol PCM_EEZ_passives:C-EU
- added R25: 10R, PCM_EEZ_passives:R_0805_2012Metric, symbol PCM_EEZ_passives:R-EU
- added R27: 1R, PCM_EEZ_passives:R_0603_1608Metric, symbol PCM_EEZ_passives:R-EU
- JP2, JP3: now left out of the parts list
- renumbered C44 to C45, C47 to C48, C48 to C49, C50 to C51, IC9 to IC10, IC10 to IC9, R25 to R29, R30 to R32, R31 to R33
Connections:
- net +VREF: now also C41.1, R25.1; no longer IC10.6 (VOUT)
- net GND: now also C41.2, R27.2
- new net: C44.1, IC10.6 (VOUT), R25.2
- new net: C44.2, R27.1
Other:
- moved on the sheet: C45, C49, IC10, Q3, R29, R32, TP2

Commit message: r4B4 (ADC replaced with ADS131A04)
Parts:
- R27: footprint PCM_EEZ_passives:R_0603_1608Metric -> PCM_EEZ_passives:R_0805_2012Metric
- renumbered C33 to C37, C34 to C38, C35 to C39, C39 to C43, C41 to C45, C44 to C48, C45 to C49, C48 to C52, C49 to C53, C51 to C55, JP2 to JP4, JP3 to JP5

Commit message: SPI channels renamed
Connections:
- net ISO_DA_MISO renamed ISO_MISO2
- net ISO_DA_MOSI renamed ISO_MOSI2
- net ISO_DA_SCLK renamed ISO_SCLK2
- net ISO_IOEXP_MISO renamed ISO_MISO1
- net ISO_IOEXP_MOSI renamed ISO_MOSI1
- net ISO_IOEXP_SCLK renamed ISO_SCLK1
Changed lines of the file:
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@@
 		)
 	)
-	(global_label "ISO_DA_MISO"
+	(global_label "ISO_MISO2"
 		(shape output)
 		(at 124.46 149.86 180)
@@
 		)
 	)
-	(global_label "ISO_IOEXP_MISO"
+	(global_label "ISO_MISO1"
 		(shape output)
 		(at 210.82 43.18 180)
@@
 		)
 	)
-	(global_label "ISO_IOEXP_SCLK"
+	(global_label "ISO_SCLK1"
 		(shape input)
 		(at 210.82 45.72 180)
@@
 		)
 		(property "Intersheetrefs" "${INTERSHEET_REFS}"
-			(at 197.9356 45.72 0)
+			(at 201.6608 45.72 0)
 			(effects
 				(font
@@
 		)
 	)
-	(global_label "ISO_DA_MOSI"
+	(global_label "ISO_MOSI2"
 		(shape input)
 		(at 27.94 43.18 180)
@@
 		)
 	)
-	(global_label "ISO_DA_SCLK"
+	(global_label "ISO_SCLK2"
 		(shape input)
 		(at 27.94 45.72 180)
@@
 		)
 	)
-	(global_label "ISO_DA_SCLK"
+	(global_label "ISO_SCLK2"
 		(shape input)
 		(at 124.46 147.32 180)
@@
 		)
 	)
-	(global_label "ISO_IOEXP_MOSI"
+	(global_label "ISO_MOSI1"
 		(shape input)
 		(at 210.82 48.26 180)
