File: KiCad/DAC_Vref_IOEXP_Temp.kicad_sch (KiCad schematic)
At the start: 34 parts, among them IC10 REF5025AIDR, IC13 PCAL9722HNMP, IC6 DAC8552IDGKR, IC7 74AUP1G74DC,125, IC9 TC77-5.0MCTTR, Q1 BSS84, Q2 BSS84, Q3 BSS84

Commit message: Move DAC to SPI channel 1
Connections:
- net ISO_MOSI2 is gone; now on net ISO_MOSI1: IC6.7 (DIN)
- net ISO_SCLK1: now also IC6.6 (SCLK)
- net ISO_SCLK2: no longer IC6.6 (SCLK)
Other:
- note added: "Requires SPI_MODE1 (CPOL=0, CPHA=1)"
- note removed: "Requires SPI_MODE1"
- moved on the sheet: C37, C38, C39, C53, IC6

Commit message: Additional 2 ch isolator added for OEP and temp sensor CS
Parts:
- removed R33: 10K, PCM_EEZ_passives:R_0805_2012Metric, symbol PCM_EEZ_passives:R-EU
- renumbered C37 to C39, C38 to C40, C39 to C41, C43 to C45, C45 to C47, C48 to C50, C49 to C51, C52 to C54, C53 to C55, C55 to C57, IC9 to IC10, IC10 to IC11, IC13 to IC14, IC6 to IC7, IC7 to IC8
Connections:
- net ISO_MISO2 is gone; now on net ISO_MISO1: IC10.4 (SI/O)
- net ISO_SCLK2 is gone; now on net ISO_SCLK1: IC10.3 (SCLK)
- net ~{ISO_IOEXP_CS}: now reaches IC14.23 (~{CS})
- net TEMP_CS: no longer names the net of IC14.10 (P1_1)
- net TEMP_CS: no longer IC10.1 (~{CS})
- new net ~{ISO_TEMP_CS}: IC10.1 (~{CS})
- no-connect marks 4 -> 5

Commit message: OE_LED signals marked as active low
Connections:
- net OE_LED_GREEN renamed ~{OE_LED_GREEN}
- net OE_LED_RED renamed ~{OE_LED_RED}
Changed lines of the file:
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@@
 	(title_block
 		(title "${project_name}")
-		(date "2025-12-17")
+		(date "2025-12-18")
 		(rev "${project_version}")
 		(company "${project_creator}")
@@
 		)
 	)
-	(label "OE_LED_RED"
+	(label "~{OE_LED_RED}"
 		(at 251.46 60.96 180)
 		(effects
@@
 		)
 	)
-	(label "OE_LED_RED"
+	(label "~{OE_LED_RED}"
 		(at 78.74 139.7 180)
 		(effects
@@
 		)
 	)
-	(label "OE_LED_GREEN"
+	(label "~{OE_LED_GREEN}"
 		(at 251.46 63.5 180)
 		(effects
@@
 		)
 	)
-	(label "OE_LED_GREEN"
+	(label "~{OE_LED_GREEN}"
 		(at 78.74 134.62 180)
 		(effects
