File: KiCad/Bias_power.kicad_sch (KiCad schematic)
At the start: 43 parts, among them IC11 TPS54060DGQ, IC12 MC79L05, IC13 MC78L05, IC14 TPS7A2033PDBVR

Commit message: r4B3 version: OE fixed, new LEDs for remote programming
Parts:
- removed JP6: ~, PCM_EEZ_SMD:JP3 shorted (0603), symbol PCM_EEZ_unsorted:JP3 shorted
- C30: renamed from C39; DigiKey 1276-2723-1-ND -> 1276-3138-1-ND; Mouser 80-C1206C225M5RECLR -> 187-CL31B225KCHSNNE; TME CL31B225KBHNNNE -> C3216X7S2A225KAB
- C31: renamed from C40; DigiKey 1276-2723-1-ND -> 1276-3138-1-ND; Mouser 80-C1206C225M5RECLR -> 187-CL31B225KCHSNNE; TME CL31B225KBHNNNE -> C3216X7S2A225KAB
- renumbered C41 to C32, C42 to C36, C43 to C37, C44 to C38, C45 to C40, C46 to C41, C47 to C43, C48 to C45, C49 to C46, C50 to C49, IC12 to IC11, IC13 to IC12, IC11 to IC8, JP5 to JP6, R24 to R19, R25 to R20, R26 to R21, R27 to R23, R28 to R26, R29 to R27, R30 to R29, R31 to R30, R32 to R31, R33 to R32
Connections:
- net V+: now also C49.2, IC14.1 (IN), IC14.3 (ON/~{OFF})
- net -9V renamed -12V
Other:
- note added: "Vin,max = +6.5 V"

Commit message: EEPROM connected to H503 I2C bus
Parts:
- renumbered JP6 to JP4, R19 to R16, R20 to R17, R21 to R18, R23 to R20, R26 to R23, R27 to R24, R29 to R26, R30 to R27, R31 to R28, R32 to R29
Changed lines of the file:
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@@
 	(title_block
 		(title "${project_name}")
-		(date "2025-12-05")
+		(date "2025-12-06")
 		(rev "${project_version}")
 		(company "${project_creator}")
@@
 		(on_board yes)
 		(dnp no)
-		(property "Reference" "R30"
+		(property "Reference" "R27"
 			(at 133.35 75.565 0)
 			(effects
@@
 			(project "EEZ DIB2 DCP426"
 				(path "/65943c0e-8943-4d2a-93dc-fb4938f73312/b522d90e-ad77-4f16-838a-4f8652a53e91"
-					(reference "R30")
+					(reference "R27")
 					(unit 1)
 				)
@@
 		(on_board yes)
 		(dnp no)
-		(property "Reference" "R27"
+		(property "Reference" "R24"
 			(at 113.03 68.58 0)
 			(effects
@@
 			(project "EEZ DIB2 DCP426"
 				(path "/65943c0e-8943-4d2a-93dc-fb4938f73312/b522d90e-ad77-4f16-838a-4f8652a53e91"
-					(reference "R27")
+					(reference "R24")
 					(unit 1)
 				)
@@
 		(on_board yes)
 		(dnp no)
-		(property "Reference" "R29"
+		(property "Reference" "R26"
 			(at 129.54 36.83 90)
 			(effects
@@
 			(project "EEZ DIB2 DCP426"
 				(path "/65943c0e-8943-4d2a-93dc-fb4938f73312/b522d90e-ad77-4f16-838a-4f8652a53e91"
-					(reference "R29")
+					(reference "R26")
 					(unit 1)
 				)
@@
 		(on_board yes)
 		(dnp no)
-		(property "Reference" "JP6"
+		(property "Reference" "JP4"
 			(at 144.78 58.42 0)
 			(effects
@@
 			(project ""
 				(path "/65943c0e-8943-4d2a-93dc-fb4938f73312/b522d90e-ad77-4f16-838a-4f8652a53e91"
-					(reference "JP6")
+					(reference "JP4")
 					(unit 1)
 				)
@@
 		(on_board yes)
 		(dnp no)
-		(property "Reference" "R20"
+		(property "Reference" "R17"
 			(at 39.37 73.025 0)
 			(effects
@@
 			(project "EEZ DIB2 DCP426"
 				(path "/65943c0e-8943-4d2a-93dc-fb4938f73312/b522d90e-ad77-4f16-838a-4f8652a53e91"
-					(reference "R20")
+					(reference "R17")
 					(unit 1)
 				)
@@
 		(on_board yes)
 		(dnp no)
-		(property "Reference" "R26"
+		(property "Reference" "R23"
 			(at 87.63 86.36 0)
 			(effects
@@
 			(project "EEZ DIB2 DCP426"
 				(path "/65943c0e-8943-4d2a-93dc-fb4938f73312/b522d90e-ad77-4f16-838a-4f8652a53e91"
-					(reference "R26")
+					(reference "R23")
 					(unit 1)
 				)
@@
 		(on_board yes)
 		(dnp no)
-		(property "Reference" "R23"
+		(property "Reference" "R20"
 			(at 48.26 77.47 90)
 			(effects
@@
 			(project "EEZ DIB2 DCP426"
 				(path "/65943c0e-8943-4d2a-93dc-fb4938f73312/b522d90e-ad77-4f16-838a-4f8652a53e91"
-					(reference "R23")
+					(reference "R20")
 					(unit 1)
 				)
@@
 		(on_board yes)
 		(dnp no)
-		(property "Reference" "R21"
+		(property "Reference" "R18"
 			(at 45.72 62.23 90)
 			(effects
@@
 			(project "EEZ DIB2 DCP426"
 				(path "/65943c0e-8943-4d2a-93dc-fb4938f73312/b522d90e-ad77-4f16-838a-4f8652a53e91"
-					(reference "R21")
+					(reference "R18")
 					(unit 1)
 				)
@@
 		(on_board yes)
 		(dnp no)
-		(property "Reference" "R19"
+		(property "Reference" "R16"
 			(at 31.75 76.2 0)
 			(effects
@@
 			(project "EEZ DIB2 DCP426"
 				(path "/65943c0e-8943-4d2a-93dc-fb4938f73312/b522d90e-ad77-4f16-838a-4f8652a53e91"
-					(reference "R19")
+					(reference "R16")
 					(unit 1)
 				)
@@
 		(on_board yes)
 		(dnp no)
-		(property "Reference" "R31"
+		(property "Reference" "R28"
 			(at 133.35 91.44 0)
 			(effects
@@
 			(project "EEZ DIB2 DCP426"
 				(path "/65943c0e-8943-4d2a-93dc-fb4938f73312/b522d90e-ad77-4f16-838a-4f8652a53e91"
-					(reference "R31")
+					(reference "R28")
 					(unit 1)
 				)
@@
 		(on_board yes)
 		(dnp no)
-		(property "Reference" "R32"
+		(property "Reference" "R29"
 			(at 139.7 62.23 90)
 			(effects
@@
 			(project "EEZ DIB2 DCP426"
 				(path "/65943c0e-8943-4d2a-93dc-fb4938f73312/b522d90e-ad77-4f16-838a-4f8652a53e91"
-					(reference "R32")
+					(reference "R29")
 					(unit 1)
 				)

Commit message: Vref tantalum capacitor removed
Parts:
- renumbered C41 to C42, C45 to C46, C46 to C47, C49 to C50, C51 to C52, C52 to C53, C53 to C54, R27 to R28, R28 to R30, R29 to R31
Changed lines of the file:
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@@
 		(on_board yes)
 		(dnp no)
-		(property "Reference" "#SUPPLY020"
+		(property "Reference" "#SUPPLY021"
 			(at 139.7 53.34 0)
 			(effects
@@
 			(project "EEZ DIB2 DCP426"
 				(path "/65943c0e-8943-4d2a-93dc-fb4938f73312/b522d90e-ad77-4f16-838a-4f8652a53e91"
-					(reference "#SUPPLY020")
+					(reference "#SUPPLY021")
 					(unit 1)
 				)
@@
 		(on_board yes)
 		(dnp no)
-		(property "Reference" "C53"
+		(property "Reference" "C54"
 			(at 244.475 109.22 0)
 			(effects
@@
 			(project "EEZ DIB2 DCP426"
 				(path "/65943c0e-8943-4d2a-93dc-fb4938f73312/b522d90e-ad77-4f16-838a-4f8652a53e91"
-					(reference "C53")
+					(reference "C54")
 					(unit 1)
 				)
@@
 		(on_board yes)
 		(dnp no)
-		(property "Reference" "R27"
+		(property "Reference" "R28"
 			(at 133.35 75.565 0)
 			(effects
@@
 			(project "EEZ DIB2 DCP426"
 				(path "/65943c0e-8943-4d2a-93dc-fb4938f73312/b522d90e-ad77-4f16-838a-4f8652a53e91"
-					(reference "R27")
+					(reference "R28")
 					(unit 1)
 				)
@@
 		(on_board yes)
 		(dnp no)
-		(property "Reference" "C41"
+		(property "Reference" "C42"
 			(at 121.92 43.18 0)
 			(effects
@@
 			(project "EEZ DIB2 DCP426"
 				(path "/65943c0e-8943-4d2a-93dc-fb4938f73312/b522d90e-ad77-4f16-838a-4f8652a53e91"
-					(reference "C41")
+					(reference "C42")
 					(unit 1)
 				)
@@
 		(on_board yes)
 		(dnp no)
-		(property "Reference" "#SUPPLY021"
+		(property "Reference" "#SUPPLY022"
 			(at 147.32 104.14 0)
 			(effects
@@
 			(project "EEZ DIB2 DCP426"
 				(path "/65943c0e-8943-4d2a-93dc-fb4938f73312/b522d90e-ad77-4f16-838a-4f8652a53e91"
-					(reference "#SUPPLY021")
+					(reference "#SUPPLY022")
 					(unit 1)
 				)
@@
 		(on_board yes)
 		(dnp no)
-		(property "Reference" "C46"
+		(property "Reference" "C47"
 			(at 150.114 77.089 0)
 			(effects
@@
 			(project "EEZ DIB2 DCP426"
 				(path "/65943c0e-8943-4d2a-93dc-fb4938f73312/b522d90e-ad77-4f16-838a-4f8652a53e91"
-					(reference "C46")
+					(reference "C47")
 					(unit 1)
 				)
@@
 		(on_board yes)
 		(dnp no)
-		(property "Reference" "#SUPPLY029"
+		(property "Reference" "#SUPPLY030"
 			(at 208.28 43.18 0)
 			(effects
@@
 			(project "EEZ DIB2 DCP426"
 				(path "/65943c0e-8943-4d2a-93dc-fb4938f73312/b522d90e-ad77-4f16-838a-4f8652a53e91"
-					(reference "#SUPPLY029")
+					(reference "#SUPPLY030")
 					(unit 1)
 				)
@@
 		(on_board yes)
 		(dnp no)
-		(property "Reference" "C49"
+		(property "Reference" "C50"
 			(at 205.105 111.76 0)
 			(effects
@@
 			(project "EEZ DIB2 DCP426"
 				(path "/65943c0e-8943-4d2a-93dc-fb4938f73312/b522d90e-ad77-4f16-838a-4f8652a53e91"
-					(reference "C49")
+					(reference "C50")
 					(unit 1)
 				)
@@
 		(on_board yes)
 		(dnp no)
-		(property "Reference" "#SUPPLY033"
+		(property "Reference" "#SUPPLY034"
 			(at 259.08 63.5 0)
 			(effects
@@
 			(project "EEZ DIB2 DCP426"
 				(path "/65943c0e-8943-4d2a-93dc-fb4938f73312/b522d90e-ad77-4f16-838a-4f8652a53e91"
-					(reference "#SUPPLY033")
+					(reference "#SUPPLY034")
 					(unit 1)
 				)
@@
 		(on_board yes)
 		(dnp no)
-		(property "Reference" "#SUPPLY032"
+		(property "Reference" "#SUPPLY033"
 			(at 243.84 121.92 0)
 			(effects
@@
 			(project "EEZ DIB2 DCP426"
 				(path "/65943c0e-8943-4d2a-93dc-fb4938f73312/b522d90e-ad77-4f16-838a-4f8652a53e91"
-					(reference "#SUPPLY032")
+					(reference "#SUPPLY033")
 					(unit 1)
 				)
@@
 		(on_board yes)
 		(dnp no)
-		(property "Reference" "C52"
+		(property "Reference" "C53"
 			(at 221.361 32.131 0)
 			(effects
@@
 			(project "EEZ DIB2 DCP426"
 				(path "/65943c0e-8943-4d2a-93dc-fb4938f73312/b522d90e-ad77-4f16-838a-4f8652a53e91"
-					(reference "C52")
+					(reference "C53")
 					(unit 1)
 				)
@@
 		(on_board yes)
 		(dnp no)
-		(property "Reference" "#SUPPLY028"
+		(property "Reference" "#SUPPLY029"
 			(at 205.74 121.92 0)
 			(effects
@@
 			(project "EEZ DIB2 DCP426"
 				(path "/65943c0e-8943-4d2a-93dc-fb4938f73312/b522d90e-ad77-4f16-838a-4f8652a53e91"
-					(reference "#SUPPLY028")
+					(reference "#SUPPLY029")
 					(unit 1)
 				)
@@
 		(on_board yes)
 		(dnp no)
-		(property "Reference" "R28"
+		(property "Reference" "R30"
 			(at 133.35 91.44 0)
 			(effects
@@
 			(project "EEZ DIB2 DCP426"
 				(path "/65943c0e-8943-4d2a-93dc-fb4938f73312/b522d90e-ad77-4f16-838a-4f8652a53e91"
-					(reference "R28")
+					(reference "R30")
 					(unit 1)
 				)
@@
 		(on_board yes)
 		(dnp no)
-		(property "Reference" "C45"
+		(property "Reference" "C46"
 			(at 141.859 44.069 0)
 			(effects
@@
 			(project "EEZ DIB2 DCP426"
 				(path "/65943c0e-8943-4d2a-93dc-fb4938f73312/b522d90e-ad77-4f16-838a-4f8652a53e91"
-					(reference "C45")
+					(reference "C46")
 					(unit 1)
 				)
@@
 		(on_board yes)
 		(dnp no)
-		(property "Reference" "#SUPPLY026"
+		(property "Reference" "#SUPPLY027"
 			(at 205.74 81.28 0)
 			(effects
@@
 			(project "EEZ DIB2 DCP426"
 				(path "/65943c0e-8943-4d2a-93dc-fb4938f73312/b522d90e-ad77-4f16-838a-4f8652a53e91"
-					(reference "#SUPPLY026")
+					(reference "#SUPPLY027")
 					(unit 1)
 				)
@@
 		(on_board yes)
 		(dnp no)
-		(property "Reference" "C51"
+		(property "Reference" "C52"
 			(at 219.075 66.04 0)
 			(effects
@@
 			(project "EEZ DIB2 DCP426"
 				(path "/65943c0e-8943-4d2a-93dc-fb4938f73312/b522d90e-ad77-4f16-838a-4f8652a53e91"
-					(reference "C51")
+					(reference "C52")
 					(unit 1)
 				)
@@
 		(on_board yes)
 		(dnp no)
-		(property "Reference" "#SUPPLY024"
+		(property "Reference" "#SUPPLY025"
 			(at 190.5 63.5 0)
 			(effects
@@
 			(project "EEZ DIB2 DCP426"
 				(path "/65943c0e-8943-4d2a-93dc-fb4938f73312/b522d90e-ad77-4f16-838a-4f8652a53e91"
-					(reference "#SUPPLY024")
+					(reference "#SUPPLY025")
 					(unit 1)
 				)
@@
 		(on_board yes)
 		(dnp no)
-		(property "Reference" "R29"
+		(property "Reference" "R31"
 			(at 139.7 62.23 90)
 			(effects
@@
 			(project "EEZ DIB2 DCP426"
 				(path "/65943c0e-8943-4d2a-93dc-fb4938f73312/b522d90e-ad77-4f16-838a-4f8652a53e91"
-					(reference "R29")
+					(reference "R31")
 					(unit 1)
 				)

Commit message: r4B4 (ADC replaced with ADS131A04)
Parts:
- FB2: renamed from FB5; value 60R@100MHz -> BLM18AG102SH1D; symbol PCM_EEZ_passives:L_EU -> PCM_EEZ_passives:L_Ferrite Bead
- FB3: renamed from FB4; value 60R@100MHz -> BLM18AG102SH1D; symbol PCM_EEZ_passives:L_EU -> PCM_EEZ_passives:L_Ferrite Bead
- renumbered C30 to C34, C31 to C35, C32 to C36, C36 to C40, C37 to C41, C38 to C42, C40 to C44, C42 to C46, C43 to C47, C46 to C50, C47 to C51, C50 to C54, C52 to C56, C53 to C57, C54 to C58, JP4 to JP6

Commit message: Additional 2 ch isolator added for OEP and temp sensor CS
Parts:
- renumbered C34 to C36, C35 to C37, C36 to C38, C40 to C42, C41 to C43, C42 to C44, C44 to C46, C46 to C48, C47 to C49, C50 to C52, C51 to C53, C54 to C56, C56 to C58, C57 to C59, C58 to C60, IC11 to IC12, IC12 to IC13, IC14 to IC15, IC8 to IC9
