File: KiCad/CC_CV_OVP.kicad_sch (KiCad schematic)
At the start: 41 parts, among them IC25 LM293D, IC26 MAX9141ESA, Q25 2N7002, Q26 2N7002, Q27 2N7002, Q28 MMBT5551, Q29 FMMT493TA, Q30 BT139B-600E, Q31 PSMN013-60YL

Commit message: r4B3 version: OE fixed, new LEDs for remote programming
Parts:
- IC25: DigiKey 296-12848-1-ND -> LM293DR2GOSCT-ND; Mouser 511-LM293DT -> 863-LM293DR2G; TME LM293D-ST -> LM293DR
- LED3: symbol PCM_EEZ_discretes:WP934MD -> PCM_EEZ_discretes:WP934MD/LYLID; DigiKey 754-2008-ND -> 350-2716-ND; LCSC (none) -> -
- R128: renamed from R127; Mouser 71-CRCW0805750RFKEB -> 71-CRCW0805750RFKEAC
- R129: renamed from R128; Mouser 71-CRCW0805750RFKEB -> 71-CRCW0805750RFKEAC
- renumbered D24 to D22, D25 to D23, JP11 to JP12, R123 to R124, R124 to R125, R125 to R126, R126 to R127, R129 to R130, R130 to R131, R131 to R132, R132 to R133, R133 to R134, R134 to R135, R135 to R136, R136 to R137, R137 to R138, R138 to R139, R139 to R140, R140 to R141, R141 to R142, R142 to R143, R143 to R144, R144 to R145

Commit message: EEPROM connected to H503 I2C bus
Parts:
- renumbered JP12 to JP10, R124 to R121, R125 to R122, R126 to R123, R127 to R124, R128 to R125, R129 to R126, R130 to R127, R131 to R128, R132 to R129, R133 to R130, R134 to R131, R135 to R132, R136 to R133, R137 to R134, R138 to R135, R139 to R136, R140 to R137, R141 to R138, R142 to R139, R143 to R140, R144 to R141, R145 to R142
Changed lines of the file:
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@@
 	(title_block
 		(title "${project_name}")
-		(date "2025-12-05")
+		(date "2025-12-06")
 		(rev "${project_version}")
 		(company "${project_creator}")
@@
 		(on_board yes)
 		(dnp no)
-		(property "Reference" "JP12"
+		(property "Reference" "JP10"
 			(at 201.295 40.64 90)
 			(effects
@@
 			(project "EEZ DIB DCP405"
 				(path "/65943c0e-8943-4d2a-93dc-fb4938f73312/5aca86d7-0c45-458c-9a52-ab1a5068ba91"
-					(reference "JP12")
+					(reference "JP10")
 					(unit 1)
 				)
@@
 		(on_board yes)
 		(dnp no)
-		(property "Reference" "R127"
+		(property "Reference" "R124"
 			(at 53.34 85.09 90)
 			(effects
@@
 			(project "EEZ DIB DCP405"
 				(path "/65943c0e-8943-4d2a-93dc-fb4938f73312/5aca86d7-0c45-458c-9a52-ab1a5068ba91"
-					(reference "R127")
+					(reference "R124")
 					(unit 1)
 				)
@@
 		(on_board yes)
 		(dnp no)
-		(property "Reference" "R134"
+		(property "Reference" "R131"
 			(at 167.64 72.39 90)
 			(effects
@@
 			(project "EEZ DIB DCP405"
 				(path "/65943c0e-8943-4d2a-93dc-fb4938f73312/5aca86d7-0c45-458c-9a52-ab1a5068ba91"
-					(reference "R134")
+					(reference "R131")
 					(unit 1)
 				)
@@
 		(on_board yes)
 		(dnp no)
-		(property "Reference" "R140"
+		(property "Reference" "R137"
 			(at 222.25 78.74 0)
 			(effects
@@
 			(project "EEZ DIB DCP405"
 				(path "/65943c0e-8943-4d2a-93dc-fb4938f73312/5aca86d7-0c45-458c-9a52-ab1a5068ba91"
-					(reference "R140")
+					(reference "R137")
 					(unit 1)
 				)
@@
 		(on_board yes)
 		(dnp no)
-		(property "Reference" "R135"
+		(property "Reference" "R132"
 			(at 176.53 57.785 0)
 			(effects
@@
 			(project "EEZ DIB DCP405"
 				(path "/65943c0e-8943-4d2a-93dc-fb4938f73312/5aca86d7-0c45-458c-9a52-ab1a5068ba91"
-					(reference "R135")
+					(reference "R132")
 					(unit 1)
 				)
@@
 		(on_board yes)
 		(dnp no)
-		(property "Reference" "R128"
+		(property "Reference" "R125"
 			(at 59.69 121.92 0)
 			(effects
@@
 			(project "EEZ DIB DCP405"
 				(path "/65943c0e-8943-4d2a-93dc-fb4938f73312/5aca86d7-0c45-458c-9a52-ab1a5068ba91"
-					(reference "R128")
+					(reference "R125")
 					(unit 1)
 				)
@@
 		(on_board yes)
 		(dnp no)
-		(property "Reference" "R131"
+		(property "Reference" "R128"
 			(at 86.36 64.77 90)
 			(effects
@@
 			(project "EEZ DIB DCP405"
 				(path "/65943c0e-8943-4d2a-93dc-fb4938f73312/5aca86d7-0c45-458c-9a52-ab1a5068ba91"
-					(reference "R131")
+					(reference "R128")
 					(unit 1)
 				)
@@
 		(on_board yes)
 		(dnp no)
-		(property "Reference" "R139"
+		(property "Reference" "R136"
 			(at 215.9 102.87 90)
 			(effects
@@
 			(project "EEZ DIB DCP405"
 				(path "/65943c0e-8943-4d2a-93dc-fb4938f73312/5aca86d7-0c45-458c-9a52-ab1a5068ba91"
-					(reference "R139")
+					(reference "R136")
 					(unit 1)
 				)
@@
 		(on_board yes)
 		(dnp no)
-		(property "Reference" "R142"
+		(property "Reference" "R139"
 			(at 242.57 50.8 0)
 			(effects
@@
 			(project "EEZ DIB DCP405"
 				(path "/65943c0e-8943-4d2a-93dc-fb4938f73312/5aca86d7-0c45-458c-9a52-ab1a5068ba91"
-					(reference "R142")
+					(reference "R139")
 					(unit 1)
 				)
@@
 		(on_board yes)
 		(dnp no)
-		(property "Reference" "R130"
+		(property "Reference" "R127"
 			(at 86.36 41.91 90)
 			(effects
@@
 			(project "EEZ DIB DCP405"
 				(path "/65943c0e-8943-4d2a-93dc-fb4938f73312/5aca86d7-0c45-458c-9a52-ab1a5068ba91"
-					(reference "R130")
+					(reference "R127")
 					(unit 1)
 				)
@@
 		(on_board yes)
 		(dnp no)
-		(property "Reference" "R144"
+		(property "Reference" "R141"
 			(at 245.11 111.125 0)
 			(effects
@@
 			(project "EEZ DIB DCP405"
 				(path "/65943c0e-8943-4d2a-93dc-fb4938f73312/5aca86d7-0c45-458c-9a52-ab1a5068ba91"
-					(reference "R144")
+					(reference "R141")
 					(unit 1)
 				)
@@
 		(on_board yes)
 		(dnp no)
-		(property "Reference" "R143"
+		(property "Reference" "R140"
 			(at 242.57 78.105 0)
 			(effects
@@
 			(project "EEZ DIB DCP405"
 				(path "/65943c0e-8943-4d2a-93dc-fb4938f73312/5aca86d7-0c45-458c-9a52-ab1a5068ba91"
-					(reference "R143")
+					(reference "R140")
 					(unit 1)
 				)
@@
 		(on_board yes)
 		(dnp no)
-		(property "Reference" "R132"
+		(property "Reference" "R129"
 			(at 86.36 82.55 90)
 			(effects
@@
 			(project "EEZ DIB DCP405"
 				(path "/65943c0e-8943-4d2a-93dc-fb4938f73312/5aca86d7-0c45-458c-9a52-ab1a5068ba91"
-					(reference "R132")
+					(reference "R129")
 					(unit 1)
 				)
@@
 		(on_board yes)
 		(dnp no)
-		(property "Reference" "R126"
+		(property "Reference" "R123"
 			(at 53.34 44.45 90)
 			(effects
@@
 			(project "EEZ DIB DCP405"
 				(path "/65943c0e-8943-4d2a-93dc-fb4938f73312/5aca86d7-0c45-458c-9a52-ab1a5068ba91"
-					(reference "R126")
+					(reference "R123")
 					(unit 1)
 				)
@@
 		(on_board yes)
 		(dnp no)
-		(property "Reference" "R125"
+		(property "Reference" "R122"
 			(at 44.45 80.645 0)
 			(effects
@@
 			(project "EEZ DIB DCP405"
 				(path "/65943c0e-8943-4d2a-93dc-fb4938f73312/5aca86d7-0c45-458c-9a52-ab1a5068ba91"
-					(reference "R125")
+					(reference "R122")
 					(unit 1)
 				)
@@
 		(on_board yes)
 		(dnp no)
-		(property "Reference" "R129"
+		(property "Reference" "R126"
 			(at 74.93 114.3 0)
 			(effects
@@
 			(project "EEZ DIB DCP405"
 				(path "/65943c0e-8943-4d2a-93dc-fb4938f73312/5aca86d7-0c45-458c-9a52-ab1a5068ba91"
-					(reference "R129")
+					(reference "R126")
 					(unit 1)
 				)
@@
 		(on_board yes)
 		(dnp no)
-		(property "Reference" "R138"
+		(property "Reference" "R135"
 			(at 215.9 62.23 90)
 			(effects
@@
 			(project "EEZ DIB DCP405"
 				(path "/65943c0e-8943-4d2a-93dc-fb4938f73312/5aca86d7-0c45-458c-9a52-ab1a5068ba91"
-					(reference "R138")
+					(reference "R135")
 					(unit 1)
 				)
@@
 		(on_board yes)
 		(dnp no)
-		(property "Reference" "R141"
+		(property "Reference" "R138"
 			(at 234.95 50.8 0)
 			(effects
@@
 			(project "EEZ DIB DCP405"
 				(path "/65943c0e-8943-4d2a-93dc-fb4938f73312/5aca86d7-0c45-458c-9a52-ab1a5068ba91"
-					(reference "R141")
+					(reference "R138")
 					(unit 1)
 				)
@@
 		(on_board yes)
 		(dnp no)
-		(property "Reference" "R137"
+		(property "Reference" "R134"
 			(at 208.28 34.29 90)
 			(effects
@@
 			(project "EEZ DIB DCP405"
 				(path "/65943c0e-8943-4d2a-93dc-fb4938f73312/5aca86d7-0c45-458c-9a52-ab1a5068ba91"
-					(reference "R137")
+					(reference "R134")
 					(unit 1)
 				)
@@
 		(on_board yes)
 		(dnp no)
-		(property "Reference" "R136"
+		(property "Reference" "R133"
 			(at 201.93 109.22 0)
 			(effects
@@
 			(project "EEZ DIB DCP405"
 				(path "/65943c0e-8943-4d2a-93dc-fb4938f73312/5aca86d7-0c45-458c-9a52-ab1a5068ba91"
-					(reference "R136")
+					(reference "R133")
 					(unit 1)
 				)
@@
 		(on_board yes)
 		(dnp no)
-		(property "Reference" "R133"
+		(property "Reference" "R130"
 			(at 167.64 49.53 90)
 			(effects
@@
 			(project "EEZ DIB DCP405"
 				(path "/65943c0e-8943-4d2a-93dc-fb4938f73312/5aca86d7-0c45-458c-9a52-ab1a5068ba91"
-					(reference "R133")
+					(reference "R130")
 					(unit 1)
 				)
@@
 		(on_board yes)
 		(dnp no)
-		(property "Reference" "R145"
+		(property "Reference" "R142"
 			(at 245.11 124.46 0)
 			(effects
@@
 			(project "EEZ DIB DCP405"
 				(path "/65943c0e-8943-4d2a-93dc-fb4938f73312/5aca86d7-0c45-458c-9a52-ab1a5068ba91"
-					(reference "R145")
+					(reference "R142")
 					(unit 1)
 				)
@@
 		(on_board yes)
 		(dnp no)
-		(property "Reference" "R124"
+		(property "Reference" "R121"
 			(at 46.99 40.005 0)
 			(effects
@@
 			(project "EEZ DIB DCP405"
 				(path "/65943c0e-8943-4d2a-93dc-fb4938f73312/5aca86d7-0c45-458c-9a52-ab1a5068ba91"
-					(reference "R124")
+					(reference "R121")
 					(unit 1)
 				)

Commit message: Vref tantalum capacitor removed
Parts:
- renumbered C116 to C117, C117 to C118, C118 to C119, C119 to C120, C120 to C121, R121 to R123, R122 to R124, R123 to R125, R124 to R126, R125 to R127, R126 to R128, R127 to R129, R128 to R130, R129 to R131, R130 to R132, R131 to R133, R132 to R134, R133 to R135, R134 to R136, R135 to R137, R136 to R138, R137 to R139, R138 to R140, R139 to R141, R140 to R142, R141 to R143, R142 to R144

Commit message: r4B4 (ADC replaced with ADS131A04)
Parts:
- renumbered C117 to C121, C118 to C122, C119 to C123, C120 to C124, C121 to C125, JP10 to JP12
Changed lines of the file:
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@@
 	(title_block
 		(title "${project_name}")
-		(date "2025-12-06")
+		(date "2025-12-07")
 		(rev "${project_version}")
 		(company "${project_creator}")
@@
 		(on_board yes)
 		(dnp no)
-		(property "Reference" "JP10"
+		(property "Reference" "JP12"
 			(at 201.295 40.64 90)
 			(effects
@@
 			(project "EEZ DIB DCP405"
 				(path "/65943c0e-8943-4d2a-93dc-fb4938f73312/5aca86d7-0c45-458c-9a52-ab1a5068ba91"
-					(reference "JP10")
+					(reference "JP12")
 					(unit 1)
 				)
@@
 		(on_board yes)
 		(dnp no)
-		(property "Reference" "C119"
+		(property "Reference" "C123"
 			(at 183.134 64.516 0)
 			(effects
@@
 			(project "EEZ DIB DCP405"
 				(path "/65943c0e-8943-4d2a-93dc-fb4938f73312/5aca86d7-0c45-458c-9a52-ab1a5068ba91"
-					(reference "C119")
+					(reference "C123")
 					(unit 1)
 				)
@@
 		(on_board yes)
 		(dnp no)
-		(property "Reference" "#SUPPLY063"
+		(property "Reference" "#SUPPLY068"
 			(at 60.96 144.78 0)
 			(effects
@@
 			(project "EEZ DIB DCP405"
 				(path "/65943c0e-8943-4d2a-93dc-fb4938f73312/5aca86d7-0c45-458c-9a52-ab1a5068ba91"
-					(reference "#SUPPLY063")
+					(reference "#SUPPLY068")
 					(unit 1)
 				)
@@
 		(on_board yes)
 		(dnp no)
-		(property "Reference" "#SUPPLY064"
+		(property "Reference" "#SUPPLY069"
 			(at 73.66 137.16 0)
 			(effects
@@
 			(project "EEZ DIB DCP405"
 				(path "/65943c0e-8943-4d2a-93dc-fb4938f73312/5aca86d7-0c45-458c-9a52-ab1a5068ba91"
-					(reference "#SUPPLY064")
+					(reference "#SUPPLY069")
 					(unit 1)
 				)
@@
 		(on_board yes)
 		(dnp no)
-		(property "Reference" "#SUPPLY065"
+		(property "Reference" "#SUPPLY070"
 			(at 127 66.04 0)
 			(effects
@@
 			(project "EEZ DIB DCP405"
 				(path "/65943c0e-8943-4d2a-93dc-fb4938f73312/5aca86d7-0c45-458c-9a52-ab1a5068ba91"
-					(reference "#SUPPLY065")
+					(reference "#SUPPLY070")
 					(unit 1)
 				)
@@
 		(on_board yes)
 		(dnp no)
-		(property "Reference" "#+3V024"
+		(property "Reference" "#+3V026"
 			(at 45.72 30.48 0)
 			(effects
@@
 			(project "EEZ DIB DCP405"
 				(path "/65943c0e-8943-4d2a-93dc-fb4938f73312/5aca86d7-0c45-458c-9a52-ab1a5068ba91"
-					(reference "#+3V024")
+					(reference "#+3V026")
 					(unit 1)
 				)
@@
 		(on_board yes)
 		(dnp no)
-		(property "Reference" "#SUPPLY066"
+		(property "Reference" "#SUPPLY071"
 			(at 175.26 66.04 0)
 			(effects
@@
 			(project "EEZ DIB DCP405"
 				(path "/65943c0e-8943-4d2a-93dc-fb4938f73312/5aca86d7-0c45-458c-9a52-ab1a5068ba91"
-					(reference "#SUPPLY066")
+					(reference "#SUPPLY071")
 					(unit 1)
 				)
@@
 		(on_board yes)
 		(dnp no)
-		(property "Reference" "#+3V025"
+		(property "Reference" "#+3V027"
 			(at 45.72 71.12 0)
 			(effects
@@
 			(project "EEZ DIB DCP405"
 				(path "/65943c0e-8943-4d2a-93dc-fb4938f73312/5aca86d7-0c45-458c-9a52-ab1a5068ba91"
-					(reference "#+3V025")
+					(reference "#+3V027")
 					(unit 1)
 				)
@@
 		(on_board yes)
 		(dnp no)
-		(property "Reference" "C117"
+		(property "Reference" "C121"
 			(at 121.539 58.039 90)
 			(effects
@@
 			(project "EEZ DIB DCP405"
 				(path "/65943c0e-8943-4d2a-93dc-fb4938f73312/5aca86d7-0c45-458c-9a52-ab1a5068ba91"
-					(reference "C117")
+					(reference "C121")
 					(unit 1)
 				)
@@
 		(on_board yes)
 		(dnp no)
-		(property "Reference" "#SUPPLY070"
+		(property "Reference" "#SUPPLY075"
 			(at 215.9 40.64 0)
 			(effects
@@
 			(project "EEZ DIB DCP405"
 				(path "/65943c0e-8943-4d2a-93dc-fb4938f73312/5aca86d7-0c45-458c-9a52-ab1a5068ba91"
-					(reference "#SUPPLY070")
+					(reference "#SUPPLY075")
 					(unit 1)
 				)
@@
 		(on_board yes)
 		(dnp no)
-		(property "Reference" "C120"
+		(property "Reference" "C124"
 			(at 190.119 41.021 90)
 			(effects
@@
 			(project "EEZ DIB DCP405"
 				(path "/65943c0e-8943-4d2a-93dc-fb4938f73312/5aca86d7-0c45-458c-9a52-ab1a5068ba91"
-					(reference "C120")
+					(reference "C124")
 					(unit 1)
 				)
@@
 		(on_board yes)
 		(dnp no)
-		(property "Reference" "#SUPPLY072"
+		(property "Reference" "#SUPPLY077"
 			(at 243.84 132.08 0)
 			(effects
@@
 			(project "EEZ DIB DCP405"
 				(path "/65943c0e-8943-4d2a-93dc-fb4938f73312/5aca86d7-0c45-458c-9a52-ab1a5068ba91"
-					(reference "#SUPPLY072")
+					(reference "#SUPPLY077")
 					(unit 1)
 				)
@@
 		(on_board yes)
 		(dnp no)
-		(property "Reference" "#SUPPLY068"
+		(property "Reference" "#SUPPLY073"
 			(at 195.58 76.2 0)
 			(effects
@@
 			(project "EEZ DIB DCP405"
 				(path "/65943c0e-8943-4d2a-93dc-fb4938f73312/5aca86d7-0c45-458c-9a52-ab1a5068ba91"
-					(reference "#SUPPLY068")
+					(reference "#SUPPLY073")
 					(unit 1)
 				)
@@
 		(on_board yes)
 		(dnp no)
-		(property "Reference" "C118"
+		(property "Reference" "C122"
 			(at 121.539 73.279 90)
 			(effects
@@
 			(project "EEZ DIB DCP405"
 				(path "/65943c0e-8943-4d2a-93dc-fb4938f73312/5aca86d7-0c45-458c-9a52-ab1a5068ba91"
-					(reference "C118")
+					(reference "C122")
 					(unit 1)
 				)
@@
 		(on_board yes)
 		(dnp no)
-		(property "Reference" "C121"
+		(property "Reference" "C125"
 			(at 193.294 107.696 0)
 			(effects
@@
 			(project "EEZ DIB DCP405"
 				(path "/65943c0e-8943-4d2a-93dc-fb4938f73312/5aca86d7-0c45-458c-9a52-ab1a5068ba91"
-					(reference "C121")
+					(reference "C125")
 					(unit 1)
 				)
@@
 		(on_board yes)
 		(dnp no)
-		(property "Reference" "#+3V026"
+		(property "Reference" "#+3V028"
 			(at 200.66 99.06 0)
 			(effects
@@
 			(project "EEZ DIB DCP405"
 				(path "/65943c0e-8943-4d2a-93dc-fb4938f73312/5aca86d7-0c45-458c-9a52-ab1a5068ba91"
-					(reference "#+3V026")
+					(reference "#+3V028")
 					(unit 1)
 				)
@@
 		(on_board yes)
 		(dnp no)
-		(property "Reference" "#SUPPLY069"
+		(property "Reference" "#SUPPLY074"
 			(at 200.66 134.62 0)
 			(effects
@@
 			(project "EEZ DIB DCP405"
 				(path "/65943c0e-8943-4d2a-93dc-fb4938f73312/5aca86d7-0c45-458c-9a52-ab1a5068ba91"
-					(reference "#SUPPLY069")
+					(reference "#SUPPLY074")
 					(unit 1)
 				)
@@
 		(on_board yes)
 		(dnp no)
-		(property "Reference" "#SUPPLY067"
+		(property "Reference" "#SUPPLY072"
 			(at 182.88 45.72 0)
 			(effects
@@
 			(project "EEZ DIB DCP405"
 				(path "/65943c0e-8943-4d2a-93dc-fb4938f73312/5aca86d7-0c45-458c-9a52-ab1a5068ba91"
-					(reference "#SUPPLY067")
+					(reference "#SUPPLY072")
 					(unit 1)
 				)
@@
 		(on_board yes)
 		(dnp no)
-		(property "Reference" "#SUPPLY071"
+		(property "Reference" "#SUPPLY076"
 			(at 223.52 88.9 0)
 			(effects
@@
 			(project "EEZ DIB DCP405"
 				(path "/65943c0e-8943-4d2a-93dc-fb4938f73312/5aca86d7-0c45-458c-9a52-ab1a5068ba91"
-					(reference "#SUPPLY071")
+					(reference "#SUPPLY076")
 					(unit 1)
 				)

Commit message: Additional 2 ch isolator added for OEP and temp sensor CS
Parts:
- renumbered C121 to C123, C122 to C124, C123 to C125, C124 to C126, C125 to C127, IC25 to IC26, IC26 to IC27, R123 to R122, R124 to R123, R125 to R124, R126 to R125, R127 to R126, R128 to R127, R129 to R128, R130 to R129, R131 to R130, R132 to R131, R133 to R132, R134 to R133, R135 to R134, R136 to R135, R137 to R136, R138 to R137, R139 to R138, R140 to R139, R141 to R140, R142 to R141, R143 to R142, R144 to R143
