File: KiCad/Power_pre-regulator.kicad_sch (KiCad schematic)
At the start: 62 parts, among them IC15 LM5145RGYR, Q4 BSC117N08NS5ATMA1, Q5 BSC039N06NSATMA1, Q6 2N7002, Q7 MMBT5401, Q8 DMP6023LFG-7, X3 B4P-VH (LF)(SN)

Commit message: r4B3 version: OE fixed, new LEDs for remote programming
Parts:
- added JP8: ~, PCM_EEZ_connectors:M22-2010246, symbol PCM_EEZ_unsorted:JP2 open 2mm THT
- added TP11: TEST-PIN_0.9MM, PCM_EEZ_THT:Testhole 24_50mils, symbol PCM_EEZ_unsorted:PCB test point
- added TP8: PCB_TEST_TABSHIELD, PCM_EEZ_THT:Testhole 24_50mils, symbol PCM_EEZ_unsorted:PCB test point
- C57: DigiKey 1276-2723-1-ND -> 1276-3138-1-ND; Mouser 80-C1206C225M5RECLR -> 187-CL31B225KCHSNNE; TME CL31B225KBHNNNE -> C3216X7S2A225KAB
- C63: Mouser 710-885012007058 -> 80-C0805C151J5G
- C67: Mouser 710-885012007040 -> 80-C0603C102K5R7040
- JP7: symbol PCM_EEZ_unsorted:JP2 open -> PCM_EEZ_unsorted:JP2 open 2mm THT; DigiKey 952-3309-ND -> M22-2010346-ND; TME ZL303-02P -> -; now in the parts list
- renumbered JP8 to JP9, R34 to R35, R35 to R36, R36 to R37, R37 to R38, R38 to R39, R39 to R40, R40 to R41, R41 to R42, R42 to R43, R43 to R44, R44 to R45, R45 to R46, R46 to R47, R47 to R48, R48 to R49, R49 to R50, TP9 to TP10, TP10 to TP12, TP8 to TP9
Connections:
- net DUTY_100: now also TP11.1 (P$1)
- net GND: now also TP8.1 (P$1)
- net OE_TRIG renamed PREG_OE
- net PREG_OE: now also JP8.2
- new net +3V3: JP8.1
Other:
- note added: "Vcc,max = +13 V"
- moved on the sheet: R35, R37, RV1

Commit message: EEPROM connected to H503 I2C bus
Parts:
- renumbered JP7 to JP5, JP8 to JP6, JP9 to JP7, R35 to R32, R36 to R33, R37 to R34, R38 to R35, R39 to R36, R40 to R37, R41 to R38, R42 to R39, R43 to R40, R44 to R41, R45 to R42, R46 to R43, R47 to R44, R48 to R45, R49 to R46, R50 to R47
Changed lines of the file:
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@@
 	(title_block
 		(title "${project_name}")
-		(date "2025-12-05")
+		(date "2025-12-06")
 		(rev "${project_version}")
 		(company "${project_creator}")
@@
 		(on_board yes)
 		(dnp no)
-		(property "Reference" "R40"
+		(property "Reference" "R37"
 			(at 147.32 90.17 90)
 			(effects
@@
 			(project "EEZ DIB DCP405"
 				(path "/65943c0e-8943-4d2a-93dc-fb4938f73312/55df2794-308a-4204-a97c-7cdafc416b78"
-					(reference "R40")
+					(reference "R37")
 					(unit 1)
 				)
@@
 		(on_board yes)
 		(dnp no)
-		(property "Reference" "R42"
+		(property "Reference" "R39"
 			(at 171.45 102.235 0)
 			(effects
@@
 			(project "EEZ DIB DCP405"
 				(path "/65943c0e-8943-4d2a-93dc-fb4938f73312/55df2794-308a-4204-a97c-7cdafc416b78"
-					(reference "R42")
+					(reference "R39")
 					(unit 1)
 				)
@@
 		(on_board yes)
 		(dnp no)
-		(property "Reference" "R47"
+		(property "Reference" "R44"
 			(at 226.06 82.55 90)
 			(effects
@@
 			(project "EEZ DIB DCP405"
 				(path "/65943c0e-8943-4d2a-93dc-fb4938f73312/55df2794-308a-4204-a97c-7cdafc416b78"
-					(reference "R47")
+					(reference "R44")
 					(unit 1)
 				)
@@
 		(on_board yes)
 		(dnp no)
-		(property "Reference" "R50"
+		(property "Reference" "R47"
 			(at 246.38 135.89 90)
 			(effects
@@
 			(project "EEZ DIB DCP405"
 				(path "/65943c0e-8943-4d2a-93dc-fb4938f73312/55df2794-308a-4204-a97c-7cdafc416b78"
-					(reference "R50")
+					(reference "R47")
 					(unit 1)
 				)
@@
 		(on_board yes)
 		(dnp yes)
-		(property "Reference" "JP8"
+		(property "Reference" "JP6"
 			(at 50.8 67.31 0)
 			(effects
@@
 			(project "EEZ DIB DCP405plus"
 				(path "/65943c0e-8943-4d2a-93dc-fb4938f73312/55df2794-308a-4204-a97c-7cdafc416b78"
-					(reference "JP8")
+					(reference "JP6")
 					(unit 1)
 				)
@@
 		(on_board yes)
 		(dnp yes)
-		(property "Reference" "R46"
+		(property "Reference" "R43"
 			(at 217.17 63.5 0)
 			(effects
@@
 			(project "EEZ DIB DCP405plus"
 				(path "/65943c0e-8943-4d2a-93dc-fb4938f73312/55df2794-308a-4204-a97c-7cdafc416b78"
-					(reference "R46")
+					(reference "R43")
 					(unit 1)
 				)
@@
 		(on_board yes)
 		(dnp no)
-		(property "Reference" "R48"
+		(property "Reference" "R45"
 			(at 229.87 121.92 0)
 			(effects
@@
 			(project "EEZ DIB DCP405"
 				(path "/65943c0e-8943-4d2a-93dc-fb4938f73312/55df2794-308a-4204-a97c-7cdafc416b78"
-					(reference "R48")
+					(reference "R45")
 					(unit 1)
 				)
@@
 		(on_board yes)
 		(dnp no)
-		(property "Reference" "R39"
+		(property "Reference" "R36"
 			(at 93.98 123.19 90)
 			(effects
@@
 			(project "EEZ DIB DCP405"
 				(path "/65943c0e-8943-4d2a-93dc-fb4938f73312/55df2794-308a-4204-a97c-7cdafc416b78"
-					(reference "R39")
+					(reference "R36")
 					(unit 1)
 				)
@@
 		(on_board yes)
 		(dnp yes)
-		(property "Reference" "R36"
+		(property "Reference" "R33"
 			(at 41.91 29.21 0)
 			(effects
@@
 			(project "EEZ DIB DCP405"
 				(path "/65943c0e-8943-4d2a-93dc-fb4938f73312/55df2794-308a-4204-a97c-7cdafc416b78"
-					(reference "R36")
+					(reference "R33")
 					(unit 1)
 				)
@@
 		(on_board yes)
 		(dnp no)
-		(property "Reference" "R45"
+		(property "Reference" "R42"
 			(at 217.17 121.92 0)
 			(effects
@@
 			(project "EEZ DIB DCP405"
 				(path "/65943c0e-8943-4d2a-93dc-fb4938f73312/55df2794-308a-4204-a97c-7cdafc416b78"
-					(reference "R45")
+					(reference "R42")
 					(unit 1)
 				)
@@
 		(on_board yes)
 		(dnp no)
-		(property "Reference" "R41"
+		(property "Reference" "R38"
 			(at 152.4 115.57 90)
 			(effects
@@
 			(project "EEZ DIB DCP405"
 				(path "/65943c0e-8943-4d2a-93dc-fb4938f73312/55df2794-308a-4204-a97c-7cdafc416b78"
-					(reference "R41")
+					(reference "R38")
 					(unit 1)
 				)
@@
 		(on_board yes)
 		(dnp no)
-		(property "Reference" "JP9"
+		(property "Reference" "JP7"
 			(at 95.885 102.87 0)
 			(effects
@@
 			(project "EEZ DIB DCP405"
 				(path "/65943c0e-8943-4d2a-93dc-fb4938f73312/55df2794-308a-4204-a97c-7cdafc416b78"
-					(reference "JP9")
+					(reference "JP7")
 					(unit 1)
 				)
@@
 		(on_board yes)
 		(dnp no)
-		(property "Reference" "R38"
+		(property "Reference" "R35"
 			(at 69.85 91.44 0)
 			(effects
@@
 			(project "EEZ DIB DCP405"
 				(path "/65943c0e-8943-4d2a-93dc-fb4938f73312/55df2794-308a-4204-a97c-7cdafc416b78"
-					(reference "R38")
+					(reference "R35")
 					(unit 1)
 				)
@@
 		(on_board yes)
 		(dnp yes)
-		(property "Reference" "R37"
+		(property "Reference" "R34"
 			(at 53.34 171.45 90)
 			(effects
@@
 			(project "EEZ DIB DCP405plus"
 				(path "/65943c0e-8943-4d2a-93dc-fb4938f73312/55df2794-308a-4204-a97c-7cdafc416b78"
-					(reference "R37")
+					(reference "R34")
 					(unit 1)
 				)
@@
 		(on_board yes)
 		(dnp no)
-		(property "Reference" "R49"
+		(property "Reference" "R46"
 			(at 236.22 135.89 90)
 			(effects
@@
 			(project "EEZ DIB DCP405"
 				(path "/65943c0e-8943-4d2a-93dc-fb4938f73312/55df2794-308a-4204-a97c-7cdafc416b78"
-					(reference "R49")
+					(reference "R46")
 					(unit 1)
 				)
@@
 		(on_board yes)
 		(dnp no)
-		(property "Reference" "R43"
+		(property "Reference" "R40"
 			(at 201.93 147.32 0)
 			(effects
@@
 			(project "EEZ DIB DCP405"
 				(path "/65943c0e-8943-4d2a-93dc-fb4938f73312/55df2794-308a-4204-a97c-7cdafc416b78"
-					(reference "R43")
+					(reference "R40")
 					(unit 1)
 				)
@@
 		(on_board yes)
 		(dnp yes)
-		(property "Reference" "R35"
+		(property "Reference" "R32"
 			(at 40.64 171.45 90)
 			(effects
@@
 			(project "EEZ DIB DCP405plus"
 				(path "/65943c0e-8943-4d2a-93dc-fb4938f73312/55df2794-308a-4204-a97c-7cdafc416b78"
-					(reference "R35")
+					(reference "R32")
 					(unit 1)
 				)
@@
 		(on_board yes)
 		(dnp yes)
-		(property "Reference" "R44"
+		(property "Reference" "R41"
 			(at 212.09 40.64 0)
 			(effects
@@
 			(project "EEZ DIB DCP405plus"
 				(path "/65943c0e-8943-4d2a-93dc-fb4938f73312/55df2794-308a-4204-a97c-7cdafc416b78"
-					(reference "R44")
+					(reference "R41")
 					(unit 1)
 				)
@@
 		(on_board yes)
 		(dnp yes)
-		(property "Reference" "JP7"
+		(property "Reference" "JP5"
 			(at 27.305 171.45 0)
 			(effects
@@
 			(project ""
 				(path "/65943c0e-8943-4d2a-93dc-fb4938f73312/55df2794-308a-4204-a97c-7cdafc416b78"
-					(reference "JP7")
+					(reference "JP5")
 					(unit 1)
 				)

Commit message: Vref tantalum capacitor removed
Parts:
- JP5, JP6: now left out of the parts list
- renumbered C54 to C55, C55 to C56, C56 to C57, C57 to C58, C58 to C59, C59 to C60, C60 to C61, C61 to C62, C62 to C63, C63 to C64, C64 to C65, C65 to C66, C66 to C67, C67 to C68, C68 to C69, C69 to C70, C70 to C71, C71 to C72, C72 to C73, C73 to C74, C74 to C75, C75 to C76, C76 to C77, C77 to C78, R32 to R34, R33 to R35, R34 to R36, R35 to R37, R36 to R38, R37 to R39, R38 to R40, R39 to R41, R40 to R42, R41 to R43, R42 to R44, R43 to R45, R44 to R46, R45 to R47, R46 to R48, R47 to R49

Commit message: r4B4 (ADC replaced with ADS131A04)
Parts:
- renumbered C55 to C59, C56 to C60, C57 to C61, C58 to C62, C59 to C63, C60 to C64, C61 to C65, C62 to C66, C63 to C67, C64 to C68, C65 to C69, C66 to C70, C67 to C71, C68 to C72, C69 to C73, C70 to C74, C71 to C75, C72 to C76, C73 to C77, C74 to C78, C75 to C79, C76 to C80, C77 to C81, C78 to C82, JP5 to JP7, JP6 to JP8, JP7 to JP9

Commit message: Additional 2 ch isolator added for OEP and temp sensor CS
Parts:
- renumbered C59 to C61, C60 to C62, C61 to C63, C62 to C64, C63 to C65, C64 to C66, C65 to C67, C66 to C68, C67 to C69, C68 to C70, C69 to C71, C70 to C72, C71 to C73, C72 to C74, C73 to C75, C74 to C76, C75 to C77, C76 to C78, C77 to C79, C78 to C80, C79 to C81, C80 to C82, C81 to C83, C82 to C84, IC15 to IC16, R34 to R33, R35 to R34, R36 to R35, R37 to R36, R38 to R37, R39 to R38, R40 to R39, R41 to R40, R42 to R41, R43 to R42, R44 to R43, R45 to R44, R46 to R45, R47 to R46, R48 to R47, R49 to R48
