File: KiCad/Rsense_protection_power_output.kicad_sch (KiCad schematic)
At the start: 63 parts, among them IC20 SN74LVC2G08DCTR, IC21 LM293D, IC22 OPA376AIDBVR, IC23 SN74LVC1G3157DCKR, IC24 SN74LVC1G3157DCKR, J1 572-0500, J2 572-0100, K1 FTR-C1GA012G-B05 or EE2-12NU-L, Q20 MMBT5551, Q21 MMBT5551, Q22 MMBT5551, Q23 MMBT5401, Q24 2N7002, X4 TBP03R1-350-03BE, X5 ZL263-20DG

Commit message: r4B3 version: OE fixed, new LEDs for remote programming
Parts:
- removed D21, D22: BAS316, PCM_EEZ_SMD:SOD-323_1P8X1P35_ONS-M, symbol PCM_EEZ_discretes:DIODE
- removed LED2: WP934MD/2LID, PCM_EEZ_THT:WP934MD_2LID, symbol PCM_EEZ_discretes:WP934MD
- added LED2: SSF-LXH340LYGID, PCM_EEZ_THT:SSF-LXH340LYGID, symbol PCM_EEZ_discretes:SSF-LXH340LYGID
- R111: renamed from R110; Mouser 71-CRCW0805750RFKEB -> 71-CRCW0805750RFKEAC
- R114: renamed from R113; Mouser 71-CRCW0805750RFKEB -> 71-CRCW0805750RFKEAC
- renumbered D23 to D21, JP9 to JP10, JP10 to JP11, R100 to R101, R101 to R102, R102 to R103, R103 to R104, R104 to R105, R105 to R106, R106 to R107, R107 to R108, R108 to R109, R109 to R110, R111 to R112, R112 to R113, R114 to R115, R115 to R116, R116 to R117, R117 to R118, R118 to R119, R119 to R120, R120 to R121, R121 to R122, R122 to R123, TP11 to TP13, TP12 to TP14
Connections:
- net +VLED: now also LED2.YA
- net at R123.2: now also LED2.YC
- net at IC20.7 (O), IC23.6 (CTRL): now also LED2.GA
- net at IC20.3 (O), IC24.6 (CTRL): now also LED2.RA
- net at R121.2: now also LED2.GC, LED2.RC
Other:
- moved on the sheet: IC23, IC24

Commit message: EEPROM connected to H503 I2C bus
Parts:
- renumbered JP10 to JP8, JP11 to JP9, R103 to R100, R104 to R101, R105 to R102, R106 to R103, R107 to R104, R108 to R105, R109 to R106, R110 to R107, R111 to R108, R112 to R109, R113 to R110, R114 to R111, R115 to R112, R116 to R113, R117 to R114, R118 to R115, R119 to R116, R120 to R117, R121 to R118, R122 to R119, R123 to R120, R101 to R98, R102 to R99
Changed lines of the file:
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@@
 	(title_block
 		(title "${project_name}")
-		(date "2025-12-05")
+		(date "2025-12-06")
 		(rev "${project_version}")
 		(company "${project_creator}")
@@
 		(on_board yes)
 		(dnp no)
-		(property "Reference" "R117"
+		(property "Reference" "R114"
 			(at 134.62 148.59 90)
 			(effects
@@
 			(project "EEZ DIB DCP405"
 				(path "/65943c0e-8943-4d2a-93dc-fb4938f73312/5ecda23e-3d86-4b9b-8d83-de3653395b33"
-					(reference "R117")
+					(reference "R114")
 					(unit 1)
 				)
@@
 		(on_board yes)
 		(dnp no)
-		(property "Reference" "R118"
+		(property "Reference" "R115"
 			(at 138.43 129.54 0)
 			(effects
@@
 			(project "EEZ DIB DCP405"
 				(path "/65943c0e-8943-4d2a-93dc-fb4938f73312/5ecda23e-3d86-4b9b-8d83-de3653395b33"
-					(reference "R118")
+					(reference "R115")
 					(unit 1)
 				)
@@
 		(on_board yes)
 		(dnp no)
-		(property "Reference" "R123"
+		(property "Reference" "R120"
 			(at 255.27 128.905 0)
 			(effects
@@
 			(project "EEZ DIB DCP405"
 				(path "/65943c0e-8943-4d2a-93dc-fb4938f73312/5ecda23e-3d86-4b9b-8d83-de3653395b33"
-					(reference "R123")
+					(reference "R120")
 					(unit 1)
 				)
@@
 		(on_board yes)
 		(dnp no)
-		(property "Reference" "JP11"
+		(property "Reference" "JP9"
 			(at 50.165 156.21 0)
 			(effects
@@
 			(project "EEZ DIB DCP405"
 				(path "/65943c0e-8943-4d2a-93dc-fb4938f73312/5ecda23e-3d86-4b9b-8d83-de3653395b33"
-					(reference "JP11")
+					(reference "JP9")
 					(unit 1)
 				)
@@
 		(on_board yes)
 		(dnp no)
-		(property "Reference" "R114"
+		(property "Reference" "R111"
 			(at 105.41 48.26 0)
 			(effects
@@
 			(project "EEZ DIB DCP405"
 				(path "/65943c0e-8943-4d2a-93dc-fb4938f73312/5ecda23e-3d86-4b9b-8d83-de3653395b33"
-					(reference "R114")
+					(reference "R111")
 					(unit 1)
 				)
@@
 		(on_board yes)
 		(dnp no)
-		(property "Reference" "R103"
+		(property "Reference" "R100"
 			(at 60.96 140.97 90)
 			(effects
@@
 			(project "EEZ DIB DCP405"
 				(path "/65943c0e-8943-4d2a-93dc-fb4938f73312/5ecda23e-3d86-4b9b-8d83-de3653395b33"
-					(reference "R103")
+					(reference "R100")
 					(unit 1)
 				)
@@
 		(on_board yes)
 		(dnp no)
-		(property "Reference" "R120"
+		(property "Reference" "R117"
 			(at 148.59 57.15 0)
 			(effects
@@
 			(project "EEZ DIB DCP405"
 				(path "/65943c0e-8943-4d2a-93dc-fb4938f73312/5ecda23e-3d86-4b9b-8d83-de3653395b33"
-					(reference "R120")
+					(reference "R117")
 					(unit 1)
 				)
@@
 		(on_board yes)
 		(dnp no)
-		(property "Reference" "R101"
+		(property "Reference" "R98"
 			(at 49.53 70.485 0)
 			(effects
@@
 			(project "EEZ DIB DCP405"
 				(path "/65943c0e-8943-4d2a-93dc-fb4938f73312/5ecda23e-3d86-4b9b-8d83-de3653395b33"
-					(reference "R101")
+					(reference "R98")
 					(unit 1)
 				)
@@
 		(on_board yes)
 		(dnp no)
-		(property "Reference" "R112"
+		(property "Reference" "R109"
 			(at 100.33 88.265 0)
 			(effects
@@
 			(project "EEZ DIB DCP405"
 				(path "/65943c0e-8943-4d2a-93dc-fb4938f73312/5ecda23e-3d86-4b9b-8d83-de3653395b33"
-					(reference "R112")
+					(reference "R109")
 					(unit 1)
 				)
@@
 		(on_board yes)
 		(dnp no)
-		(property "Reference" "R111"
+		(property "Reference" "R108"
 			(at 100.33 73.66 0)
 			(effects
@@
 			(project "EEZ DIB DCP405"
 				(path "/65943c0e-8943-4d2a-93dc-fb4938f73312/5ecda23e-3d86-4b9b-8d83-de3653395b33"
-					(reference "R111")
+					(reference "R108")
 					(unit 1)
 				)
@@
 		(on_board yes)
 		(dnp no)
-		(property "Reference" "R104"
+		(property "Reference" "R101"
 			(at 60.96 156.21 90)
 			(effects
@@
 			(project "EEZ DIB DCP405"
 				(path "/65943c0e-8943-4d2a-93dc-fb4938f73312/5ecda23e-3d86-4b9b-8d83-de3653395b33"
-					(reference "R104")
+					(reference "R101")
 					(unit 1)
 				)
@@
 		(on_board yes)
 		(dnp no)
-		(property "Reference" "R116"
+		(property "Reference" "R113"
 			(at 109.22 148.59 90)
 			(effects
@@
 			(project "EEZ DIB DCP405"
 				(path "/65943c0e-8943-4d2a-93dc-fb4938f73312/5ecda23e-3d86-4b9b-8d83-de3653395b33"
-					(reference "R116")
+					(reference "R113")
 					(unit 1)
 				)
@@
 		(on_board yes)
 		(dnp no)
-		(property "Reference" "R115"
+		(property "Reference" "R112"
 			(at 109.22 62.23 90)
 			(effects
@@
 			(project "EEZ DIB DCP405"
 				(path "/65943c0e-8943-4d2a-93dc-fb4938f73312/5ecda23e-3d86-4b9b-8d83-de3653395b33"
-					(reference "R115")
+					(reference "R112")
 					(unit 1)
 				)
@@
 		(on_board yes)
 		(dnp no)
-		(property "Reference" "R113"
+		(property "Reference" "R110"
 			(at 105.41 33.02 0)
 			(effects
@@
 			(project "EEZ DIB DCP405"
 				(path "/65943c0e-8943-4d2a-93dc-fb4938f73312/5ecda23e-3d86-4b9b-8d83-de3653395b33"
-					(reference "R113")
+					(reference "R110")
 					(unit 1)
 				)
@@
 		(on_board yes)
 		(dnp no)
-		(property "Reference" "R121"
+		(property "Reference" "R118"
 			(at 195.58 130.81 90)
 			(effects
@@
 			(project "EEZ DIB DCP405"
 				(path "/65943c0e-8943-4d2a-93dc-fb4938f73312/5ecda23e-3d86-4b9b-8d83-de3653395b33"
-					(reference "R121")
+					(reference "R118")
 					(unit 1)
 				)
@@
 		(on_board yes)
 		(dnp no)
-		(property "Reference" "R110"
+		(property "Reference" "R107"
 			(at 96.52 62.23 90)
 			(effects
@@
 			(project "EEZ DIB DCP405"
 				(path "/65943c0e-8943-4d2a-93dc-fb4938f73312/5ecda23e-3d86-4b9b-8d83-de3653395b33"
-					(reference "R110")
+					(reference "R107")
 					(unit 1)
 				)
@@
 		(on_board yes)
 		(dnp no)
-		(property "Reference" "R107"
+		(property "Reference" "R104"
 			(at 77.47 45.72 0)
 			(effects
@@
 			(project "EEZ DIB DCP405"
 				(path "/65943c0e-8943-4d2a-93dc-fb4938f73312/5ecda23e-3d86-4b9b-8d83-de3653395b33"
-					(reference "R107")
+					(reference "R104")
 					(unit 1)
 				)
@@
 		(on_board yes)
 		(dnp no)
-		(property "Reference" "R119"
+		(property "Reference" "R116"
 			(at 143.51 129.54 0)
 			(effects
@@
 			(project "EEZ DIB DCP405"
 				(path "/65943c0e-8943-4d2a-93dc-fb4938f73312/5ecda23e-3d86-4b9b-8d83-de3653395b33"
-					(reference "R119")
+					(reference "R116")
 					(unit 1)
 				)
@@
 		(on_board yes)
 		(dnp no)
-		(property "Reference" "R102"
+		(property "Reference" "R99"
 			(at 57.15 43.18 0)
 			(effects
@@
 			(project "EEZ DIB DCP405"
 				(path "/65943c0e-8943-4d2a-93dc-fb4938f73312/5ecda23e-3d86-4b9b-8d83-de3653395b33"
-					(reference "R102")
+					(reference "R99")
 					(unit 1)
 				)
@@
 		(on_board yes)
 		(dnp no)
-		(property "Reference" "R106"
+		(property "Reference" "R103"
 			(at 69.85 86.36 0)
 			(effects
@@
 			(project "EEZ DIB DCP405"
 				(path "/65943c0e-8943-4d2a-93dc-fb4938f73312/5ecda23e-3d86-4b9b-8d83-de3653395b33"
-					(reference "R106")
+					(reference "R103")
 					(unit 1)
 				)
@@
 		(on_board yes)
 		(dnp no)
-		(property "Reference" "JP10"
+		(property "Reference" "JP8"
 			(at 50.8 140.97 0)
 			(effects
@@
 			(project "EEZ DIB DCP405"
 				(path "/65943c0e-8943-4d2a-93dc-fb4938f73312/5ecda23e-3d86-4b9b-8d83-de3653395b33"
-					(reference "JP10")
+					(reference "JP8")
 					(unit 1)
 				)
@@
 		(on_board yes)
 		(dnp no)
-		(property "Reference" "R122"
+		(property "Reference" "R119"
 			(at 250.19 149.86 0)
 			(effects
@@
 			(project "EEZ DIB DCP405"
 				(path "/65943c0e-8943-4d2a-93dc-fb4938f73312/5ecda23e-3d86-4b9b-8d83-de3653395b33"
-					(reference "R122")
+					(reference "R119")
 					(unit 1)
 				)
@@
 		(on_board yes)
 		(dnp no)
-		(property "Reference" "R105"
+		(property "Reference" "R102"
 			(at 69.85 69.85 0)
 			(effects
@@
 			(project "EEZ DIB DCP405"
 				(path "/65943c0e-8943-4d2a-93dc-fb4938f73312/5ecda23e-3d86-4b9b-8d83-de3653395b33"
-					(reference "R105")
+					(reference "R102")
 					(unit 1)
 				)
@@
 		(on_board yes)
 		(dnp no)
-		(property "Reference" "R108"
+		(property "Reference" "R105"
 			(at 93.98 135.89 90)
 			(effects
@@
 			(project "EEZ DIB DCP405"
 				(path "/65943c0e-8943-4d2a-93dc-fb4938f73312/5ecda23e-3d86-4b9b-8d83-de3653395b33"
-					(reference "R108")
+					(reference "R105")
 					(unit 1)
 				)
@@
 		(on_board yes)
 		(dnp no)
-		(property "Reference" "R109"
+		(property "Reference" "R106"
 			(at 93.98 161.29 90)
 			(effects
@@
 			(project "EEZ DIB DCP405"
 				(path "/65943c0e-8943-4d2a-93dc-fb4938f73312/5ecda23e-3d86-4b9b-8d83-de3653395b33"
-					(reference "R109")
+					(reference "R106")
 					(unit 1)
 				)

Commit message: Vref tantalum capacitor removed
Parts:
- renumbered C103 to C104, C104 to C105, C105 to C106, C106 to C107, C107 to C108, C108 to C109, C109 to C110, C110 to C111, C111 to C112, C112 to C113, C113 to C114, C114 to C115, C115 to C116, R98 to R100, R99 to R101, R100 to R102, R101 to R103, R102 to R104, R103 to R105, R104 to R106, R105 to R107, R106 to R108, R107 to R109, R108 to R110, R109 to R111, R110 to R112, R111 to R113, R112 to R114, R113 to R115, R114 to R116, R115 to R117, R116 to R118, R117 to R119, R118 to R120, R119 to R121, R120 to R122

Commit message: r4B4 (ADC replaced with ADS131A04)
Parts:
- R119: value 1R 0.1% -> 1R; footprint PCM_EEZ_passives:R_1206_3216Metric -> PCM_EEZ_passives:R_0805_2012Metric; DigiKey 1712-CPF1206B1R0E1CT-ND -> (none); LCSC C4106088 -> (none); Mouser 279-CPF1206B1R0E1 -> (none)
- renumbered C104 to C108, C105 to C109, C106 to C110, C107 to C111, C108 to C112, C109 to C113, C110 to C114, C111 to C115, C112 to C116, C113 to C117, C114 to C118, C115 to C119, C116 to C120, JP8 to JP10, JP9 to JP11

Commit message: Additional 2 ch isolator added for OEP and temp sensor CS
Parts:
- renumbered C108 to C110, C109 to C111, C110 to C112, C111 to C113, C112 to C114, C113 to C115, C114 to C116, C115 to C117, C116 to C118, C117 to C119, C118 to C120, C119 to C121, C120 to C122, IC20 to IC21, IC21 to IC22, IC22 to IC23, IC23 to IC24, IC24 to IC25, R101 to R100, R102 to R101, R103 to R102, R104 to R103, R105 to R104, R106 to R105, R107 to R106, R108 to R107, R109 to R108, R110 to R109, R111 to R110, R112 to R111, R113 to R112, R114 to R113, R115 to R114, R116 to R115, R117 to R116, R118 to R117, R119 to R118, R120 to R119, R121 to R120, R122 to R121, R100 to R99
